Commit message: Sync femur STEP exports with motor-mount feature; update PETG-CF mass/inertia
Re-export femur_left/right.step to capture the mirrored motor-mount
feature added to the femur bracket, and recompute femur mass/inertia
from the updated solid volume (density-based, PETG-CF 1.25 g/cm3).
Net mass change is negligible (~0.001%); hip_pitch/knee bore spacing
is unchanged so no joint origins were affected.

File: src/model/urdf/robot.urdf (robot description, URDF)
Before this commit: robot urdf, 28 links, 27 joints
Links:
- link femur__configuration_left: mass 0.0172732 -> 0.017273
- link femur__configuration_right: mass 0.0172732 -> 0.017273
