Commit message: Update foot mesh and mass properties for new sole geometry
The sole / ground-contact shape of the foot part was revised in CAD.
This reflects that change through the export and URDF pipeline:

- Re-exported cad/step/foot.step and cad/stl/foot.stl from the current
  Fusion geometry (shared by both foot and foot_2 links, mirrored via
  joint placement, so a single mesh pair covers both feet).
- Recomputed the foot/foot_2 <inertial> block (mass, COM, inertia
  tensor) for the new shape. Method: read the foot body's mass
  properties (COM, inertia about origin) directly from Fusion in
  world space, combined with the 8 mounting screws' world positions,
  then converted into the foot link's own local frame by walking the
  actual URDF joint chain (hip yaw/roll/pitch, knee, ankle pitch/roll)
  and composing the rotation/translation at zero configuration -- this
  avoids assuming the link frame is world-aligned, which it is not for
  this chain.
- Mass note: Fusion reports this body's (and every other structural
  body's) material as generic steel, which is clearly not the actual
  3D-printed PLA part -- this looks like an unused placeholder rather
  than a real material assignment, project-wide. Cross-checking the
  committed masses of shoulder/shoulder_2 and femur__configuration_*
  against their CAD volumes implies an effective printed density of
  roughly 1.02-1.06 g/cm^3 (below solid-PLA's 1.24, consistent with
  typical infill). Used the average (~1.044 g/cm^3) for the new foot
  body mass. This is a considered estimate, not a measurement --
  please re-weigh the printed part once available and correct if it
  differs meaningfully. The 8 M2x6 mounting screws keep their
  Fusion-reported (steel) mass, which is realistic for actual steel
  fasteners.
- Corrected right_foot_frame / left_foot_frame: with the new, thinner
  sole, the existing fixed-frame origin sat about 3.5mm above the
  actual ground-contact plane. Shifted it down to match the new sole
  surface height; the X/Y placement was checked against the new sole
  footprint and still falls comfortably inside it, so left unchanged.

Not included here: cad/step/trunk_top.step is also locally modified
relative to HEAD (unrelated to this foot change, likely from earlier
battery-compartment work) -- left untouched pending its own review.
docs/printing.md's foot photo is a static uploaded image and will now
be stale; only the user can re-capture and re-upload that.

Co-Authored-By: Claude Sonnet 5 <noreply@anthropic.com>
Claude-Session: https://claude.ai/code/session_0122vqQiRGmFNNwgYCePnSBu

File: src/model/urdf/robot.urdf (robot description, URDF)
Before this commit: robot urdf, 28 links, 27 joints
Links:
- link foot: mass 0.016823 -> 0.0271664
- link foot_2: mass 0.016823 -> 0.0271664
Joints:
- joint left_foot_frame: origin xyz=-0 -0.023 0.042 rpy=-1.5708 -1.5708 0 -> xyz=-0 -0.0265 0.042 rpy=-1.5708 -1.5708 0
- joint right_foot_frame: origin xyz=-0 -0.023 0.042 rpy=-1.5708 -1.5708 0 -> xyz=-0 -0.0265 0.042 rpy=-1.5708 -1.5708 0

Commit message: Align hip yaw axis above hip pitch axis; update PETG-CF inertia
Split the hip component and relocated the yaw/disc side by 17.5mm
(a balanced compromise between the right side's exact 18.5mm need and
the left side's 16.5mm need) so the hip yaw axis sits directly above
the hip pitch axis. The disc/yaw-mount stays mated to the trunk via a
compensating occurrence-transform shift; the roll-mount side moves by
the corresponding amount, updating right_hip_roll/left_hip_roll joint
origins in the URDF. hip_yaw origins are unchanged.

Recomputed hip/hip_2 <inertial> blocks using the new PETG-CF filament
density (1.25 g/cm3) instead of the old PLA/15%-infill convention,
composing the printed body with its 12 steel screws per side via the
parallel-axis theorem.

Re-exported cad/step/hip.step and cad/stl/hip.stl from the updated
Fusion geometry.

Co-Authored-By: Claude Sonnet 5 <noreply@anthropic.com>
Claude-Session: https://claude.ai/code/session_0122vqQiRGmFNNwgYCePnSBu

File: src/model/urdf/robot.urdf (robot description, URDF)
Before this commit: robot urdf, 28 links, 27 joints
Links:
- link hip: mass 0.00884451 -> 0.0139732
- link hip_2: mass 0.00884451 -> 0.0139732
Joints:
- joint left_hip_roll: origin xyz=0.02 0 -0.0214 rpy=-1.5708 -0 1.5708 -> xyz=0.0375 0 -0.0214 rpy=-1.5708 -0 1.5708
- joint right_hip_roll: origin xyz=-0.02 0 -0.0214 rpy=-1.5708 -0 -1.5708 -> xyz=-0.0375 0 -0.0214 rpy=-1.5708 -0 -1.5708

Commit message: Fix right/left_hip_roll origin and update PETG-CF mass/inertia for 8 links
hip_roll origin x was stale relative to commit 90fb138 ("Close 17.5mm gap
between hip roll-mount flange and hip_block free horn"), which changed
hip.step after the URDF was last regenerated (1b83c72). The joint's
rotation axis maps to local +X in the hip frame, so the 17.5mm closure
reduces |x| from 37.5mm to 20mm on both sides.

Also updates mass/inertia for the links that map 1:1 to a single printed
PETG-CF part plus only small screws (foot, femur, shoulder, hip and their
mirrored pairs), using solid-body volume from Fusion times 1.25 g/cm3
and scaling the existing inertia tensor by the same mass ratio (COM
unchanged). Links whose mass bundles a servo or bearing hardware (hip_block,
ankle_block, humerus, roll_pitch_link, camera_cover, radius, trunk) are
intentionally left untouched pending manual mass separation.

Co-Authored-By: Claude Sonnet 5 <noreply@anthropic.com>
Claude-Session: https://claude.ai/code/session_0122vqQiRGmFNNwgYCePnSBu

File: src/model/urdf/robot.urdf (robot description, URDF)
Before this commit: robot urdf, 28 links, 27 joints
Links:
- link femur__configuration_left: mass 0.014726 -> 0.0172732
- link femur__configuration_right: mass 0.014726 -> 0.0172732
- link foot: mass 0.0271664 -> 0.0301617
- link foot_2: mass 0.0271664 -> 0.0301617
- link hip: mass 0.0139732 -> 0.0097555
- link hip_2: mass 0.0139732 -> 0.0097555
- link shoulder: mass 0.00898451 -> 0.0109729
- link shoulder_2: mass 0.00898451 -> 0.0109729
Joints:
- joint left_hip_roll: origin xyz=0.0375 0 -0.0214 rpy=-1.5708 -0 1.5708 -> xyz=0.02 0 -0.0214 rpy=-1.5708 -0 1.5708
- joint right_hip_roll: origin xyz=-0.0375 0 -0.0214 rpy=-1.5708 -0 -1.5708 -> xyz=-0.02 0 -0.0214 rpy=-1.5708 -0 -1.5708

Commit message: Fix head link mass/inertia using real servo mass instead of stale composite value
The 'head' link bundles roll_servo_cradle (now PETG-CF) and an XL330
neck servo. Its old mass (174.049g) did not correspond to either the
bracket's real volume or the servo's real spec mass, so rather than
scale it by a ratio, this rebuilds it from real values: 8.834g
(roll_servo_cradle, solid PETG-CF from Fusion volume) + 18g (XL330-M288-T
datasheet mass) = 26.834g. Inertia is scaled from the old tensor by the
resulting mass ratio as an approximation; COM is left unchanged.

Co-Authored-By: Claude Sonnet 5 <noreply@anthropic.com>
Claude-Session: https://claude.ai/code/session_0122vqQiRGmFNNwgYCePnSBu

File: src/model/urdf/robot.urdf (robot description, URDF)
Before this commit: robot urdf, 28 links, 27 joints
Links:
- link head: mass 0.174049 -> 0.0268341

Commit message: Tighten neck roll/pitch and hip roll joint limits; add camera PCB mesh
Update robot.urdf joint limits to user-specified ranges:
- neck_roll: +/-45deg -> +/-25deg
- neck_pitch: +/-45deg -> -90deg (up) / +25deg (down), matching the
  sign convention of robot.xml's neck_pitch (Ry(+) tilts local +X to -Z)
- right/left_hip_roll: +/-35deg -> +/-25deg

Also add the ELP-3DGS1200P01-H120 stereo camera PCB mesh to the MJCF
assets, alongside the other exported part meshes.

Co-Authored-By: Claude Opus 5 (1M context) <noreply@anthropic.com>

File: src/model/urdf/robot.urdf (robot description, URDF)
Before this commit: robot urdf, 28 links, 27 joints
Joints:
- joint left_hip_roll: limit lower=-0.610865 upper=0.610865 effort=10 velocity=10 -> lower=-0.436332 upper=0.436332 effort=10 velocity=10
- joint neck_pitch: limit lower=-0.785398 upper=0.785398 effort=10 velocity=10 -> lower=-1.570796 upper=0.436332 effort=10 velocity=10
- joint neck_roll: limit lower=-0.785398 upper=0.785398 effort=10 velocity=10 -> lower=-0.436332 upper=0.436332 effort=10 velocity=10
- joint right_hip_roll: limit lower=-0.610865 upper=0.610865 effort=10 velocity=10 -> lower=-0.436332 upper=0.436332 effort=10 velocity=10

Commit message: Fix neck/hip mesh alignment and joint origins from live CAD; add neck servo meshes
Applied to both robot.urdf and robot.mjcf, verified against the live
Fusion 360 model on 2026-09-21 (all 21 joint axes and 69/70 mesh
placements now agree to 0.000mm):

- Add visual meshes for the 2 neck servo instances (xl330_without_horn
  in head and in roll_pitch_link), previously omitted.
- Fix head yaw axis: sat 15mm behind the real CAD servo axis.
- Fix neck_pitch axis (camera_cover body origin): sat 5mm below the
  real CAD servo axis. The camera_cover mesh itself was already
  correct; only the axis was off, matching the "cover looks right but
  the neck axis is a bit low" report.
- Fix roll_pitch_link/pitch_servo_cradle mesh Z offset (+5mm), a
  separate error from the axis fix above.
- Shift hip link and everything below it (hip_block, femur, tibia,
  ankle_block, foot) back 17.5mm in world X to match a root-level
  occurrence offset in Fusion that had never been picked up.
- Update joint limits: neck_roll +/-25deg, neck_pitch -90deg (up) /
  +25deg (down), left/right_hip_roll +/-25deg.

Co-Authored-By: Claude Sonnet 5 <noreply@anthropic.com>

File: src/model/urdf/robot.urdf (robot description, URDF)
Before this commit: robot urdf, 28 links, 27 joints
Joints:
- joint camera_left_frame: origin xyz=0.040002 0.017008 0.00503 rpy=0 0 0 -> xyz=0.040002 0.017008 0.00003 rpy=0 0 0
- joint camera_right_frame: origin xyz=0.040002 -0.042008 0.004979 rpy=0 0 0 -> xyz=0.040002 -0.042008 -2.1e-05 rpy=0 0 0
- joint head: origin xyz=-0.00204165 -0 0.126 rpy=0 0 1.5708 -> xyz=0.01295835 0 0.126 rpy=0 0 1.5708
- joint left_hip_roll: origin xyz=0.02 0 -0.0214 rpy=-1.5708 -0 1.5708 -> xyz=0.0375 0 -0.0214 rpy=-1.5708 -0 1.5708
- joint neck_pitch: origin xyz=0.0574 0.0125 -0.005 rpy=0 0 0 -> xyz=0.0574 0.0125 0 rpy=0 0 0
- joint neck_roll: origin xyz=0 0.0424 0.0225 rpy=0 0 -1.5708 -> xyz=0 0.0574 0.0225 rpy=0 0 -1.5708
- joint right_hip_roll: origin xyz=-0.02 0 -0.0214 rpy=-1.5708 -0 -1.5708 -> xyz=-0.0375 0 -0.0214 rpy=-1.5708 -0 -1.5708

Commit message: Recompute all link mass/inertia from live CAD; update battery model
All links in both robot.urdf and robot.xml recomputed 2026-09-21 from
the live Fusion 360 model, on a documented basis (see the new header
comment in each file):

- Printed parts and electronics envelopes: CAD volume x 1.25 g/cm3
  (PETG-CF, 100% infill).
- Servos: 23g each (XC330-T288-T per the ROBOTIS e-manual), replacing
  the previous 18g XL330-M288-T figure.
- Battery: 145g flat for the 3x 18650 pack (effective 1.496 g/cm3 over
  the 96.92 cm3 CAD envelope). The CAD battery box grew from a 2-cell
  (41.0mm wide) to a 3-cell (61.0 x 76.3 x 21.0mm) pack, so
  assets/battery.stl was regenerated to match.
- Screws, shims, washers and DC15 idler dummies remain massless, per
  this file's existing convention (~95g of hardware omitted
  robot-wide).

Each link's mass, COM and inertia tensor were assembled from per-part
CAD mass properties via the parallel axis theorem, so robot.urdf and
robot.xml now carry identical values.

Co-Authored-By: Claude Sonnet 5 <noreply@anthropic.com>

File: src/model/urdf/robot.urdf (robot description, URDF)
Before this commit: robot urdf, 28 links, 27 joints
Links:
- link ankle_block__configuration_left: mass 0.04722 -> 0.0577288
- link ankle_block__configuration_right: mass 0.04722 -> 0.0577288
- link camera_cover: mass 0.164569 -> 0.0360838
- link foot: mass 0.0301617 -> 0.0301613
- link foot_2: mass 0.0301617 -> 0.0301613
- link head: mass 0.0268341 -> 0.0318353
- link hip: mass 0.0097555 -> 0.00975549
- link hip_2: mass 0.0097555 -> 0.00975549
- link hip_block__configuration_left: mass 0.04763 -> 0.0583697
- link hip_block__configuration_right: mass 0.04763 -> 0.0583697
- link humerus__configuration_left: mass 0.0416867 -> 0.0514058
- link humerus__configuration_right: mass 0.0416867 -> 0.0514058
- link radius: mass 0.0115415 -> 0.0274072
- link radius_2: mass 0.0115415 -> 0.0274072
- link roll_pitch_link: mass 0.274706 -> 0.036182
- link shoulder: mass 0.0109729 -> 0.0109724
- link shoulder_2: mass 0.0109729 -> 0.0109724
- link tibia__configuration_left: mass 0.0300463 -> 0.0350657
- link tibia__configuration_right: mass 0.0300463 -> 0.0350657
- link trunk: mass 0.347283 -> 0.435626

Commit message: Add collision geometry to URDF; rebuild foot sole collision from live CAD
robot.urdf previously carried no <collision> elements at all. It now
mirrors every collision primitive already defined in robot.xml
(trunk/pelvis, radius, hip_dbl_block, femur, tibia, ankle_dbl_block,
foot), converting MuJoCo quaternions to URDF rpy and doubling MJCF's
half-extents to URDF's full box/cylinder sizes.

The foot sole collision (both files) is rebuilt from the live CAD to
match the new foot geometry, whose sole size and shape changed from
the previous revision. The sole is a single flat face whose outer
edge sits exactly on the mesh's true boundary; it's approximated by 6
nested boxes forming an inscribed staircase of the (roughly circular)
outline, covering 97.7% of its area with a max radial deficit of
1.17mm. This replaces the old 90x45mm flat-rectangle assumption.

Verified: both files parse and robot.xml loads cleanly in MuJoCo;
independently recomputed the quaternion-to-rpy conversion for every
non-foot collision primitive and it matches this diff exactly; the
new sole boxes' outer face is confirmed flush against the foot
mesh's actual boundary vertices.

Co-Authored-By: Claude Sonnet 5 <noreply@anthropic.com>

File: src/model/urdf/robot.urdf (robot description, URDF)
Before this commit: robot urdf, 28 links, 27 joints
Links:
- link ankle_block__configuration_left: geometry collision box size=0.027 0.0505 0.0125
- link ankle_block__configuration_right: geometry collision box size=0.027 0.0505 0.0125
- link femur__configuration_left: geometry collision box size=0.0025 0.018 0.01787; collision box size=0.0025 0.018 0.024941
- link femur__configuration_right: geometry collision box size=0.0025 0.018 0.01787; collision box size=0.0025 0.018 0.024941
- link foot: geometry collision box size=0.04996 0.04 0.0025; collision box size=0.0523 0.0368878 0.0025
- link foot_2: geometry collision box size=0.04996 0.04 0.0025; collision box size=0.0523 0.0368878 0.0025
- link hip_block__configuration_left: geometry collision box size=0.027 0.0505 0.0125
- link hip_block__configuration_right: geometry collision box size=0.027 0.0505 0.0125
- link radius: geometry collision cylinder length=0.016 radius=0.00525; collision cylinder length=0.0335 radius=0.009
- link radius_2: geometry collision cylinder length=0.016 radius=0.00525; collision cylinder length=0.0335 radius=0.009
- link tibia__configuration_left: geometry collision box size=0.0025 0.018 0.0165; collision box size=0.0025 0.018 0.023
- link tibia__configuration_right: geometry collision box size=0.0025 0.018 0.0165; collision box size=0.0025 0.018 0.023
- link trunk: geometry collision box size=0.058 0.066 0.0855; collision box size=0.108 0.016 0.1075

Commit message: Upgrade to XC330-T288-T servos, a 3S battery and a 2-DOF neck with a stereo camera
Redesigned printed parts (PETG-CF), a roll + pitch neck (IDs 52, 53)
carrying an ELP-3DGS1200P01-H120 stereo camera, the CAD, MJCF/URDF with
CAD mass properties and collision shapes, the BOM and assembly notes,
and the XC330 actuator constants from the identification. The simulator
uses the identified XC330 model.

Co-Authored-By: Claude Opus 5.5 (1M context) <noreply@anthropic.com>

File: src/model/urdf/robot.urdf (robot description, URDF)
Before this commit: robot urdf, 24 links, 23 joints
Links:
- added link camera_cover, mass 0.0360838
- added link camera_left, mass 1e-9
- added link camera_right, mass 1e-9
- added link roll_pitch_link, mass 0.036182
- link ankle_block__configuration_left: mass 0.04722 -> 0.0577288; geometry collision box size=0.027 0.0505 0.0125
- link ankle_block__configuration_right: mass 0.04722 -> 0.0577288; geometry collision box size=0.027 0.0505 0.0125
- link femur__configuration_left: mass 0.014726 -> 0.017273; geometry collision box size=0.0025 0.018 0.01787; collision box size=0.0025 0.018 0.024941
- link femur__configuration_right: mass 0.014726 -> 0.017273; geometry collision box size=0.0025 0.018 0.01787; collision box size=0.0025 0.018 0.024941
- link foot: mass 0.016823 -> 0.0301613; geometry collision box size=0.04996 0.04 0.0025; collision box size=0.0523 0.0368878 0.0025
- link foot_2: mass 0.016823 -> 0.0301613; geometry collision box size=0.04996 0.04 0.0025; collision box size=0.0523 0.0368878 0.0025
- link head: mass 0.0166215 -> 0.0318353
- link hip: mass 0.00884451 -> 0.00975549
- link hip_2: mass 0.00884451 -> 0.00975549
- link hip_block__configuration_left: mass 0.04763 -> 0.0583697; geometry collision box size=0.027 0.0505 0.0125
- link hip_block__configuration_right: mass 0.04763 -> 0.0583697; geometry collision box size=0.027 0.0505 0.0125
- link humerus__configuration_left: mass 0.0416867 -> 0.0514058
- link humerus__configuration_right: mass 0.0416867 -> 0.0514058
- link radius: mass 0.0115415 -> 0.0274072; geometry collision cylinder length=0.016 radius=0.00525; collision cylinder length=0.0335 radius=0.009
- link radius_2: mass 0.0115415 -> 0.0274072; geometry collision cylinder length=0.016 radius=0.00525; collision cylinder length=0.0335 radius=0.009
- link shoulder: mass 0.00898451 -> 0.0109724
- link shoulder_2: mass 0.00898451 -> 0.0109724
- link tibia__configuration_left: mass 0.0300463 -> 0.0350657; geometry collision box size=0.0025 0.018 0.0165; collision box size=0.0025 0.018 0.023
- link tibia__configuration_right: mass 0.0300463 -> 0.0350657; geometry collision box size=0.0025 0.018 0.0165; collision box size=0.0025 0.018 0.023
- link trunk: mass 0.347283 -> 0.435626; geometry collision box size=0.058 0.066 0.0855; collision box size=0.108 0.016 0.1075
Joints:
- added joint camera_left_frame: type fixed, parent camera_cover, child camera_left, origin xyz=0.040002 0.017008 0.00003 rpy=0 0 0, axis 0 0 0
- added joint camera_right_frame: type fixed, parent camera_cover, child camera_right, origin xyz=0.040002 -0.042008 -2.1e-05 rpy=0 0 0, axis 0 0 0
- added joint neck_pitch: type revolute, parent roll_pitch_link, child camera_cover, origin xyz=0.0574 0.0125 0 rpy=0 0 0, axis 0 1 0, limit lower=-1.570796 upper=0.436332 effort=10 velocity=10
- added joint neck_roll: type revolute, parent head, child roll_pitch_link, origin xyz=0 0.0574 0.0225 rpy=0 0 -1.5708, axis 1 0 0, limit lower=-0.436332 upper=0.436332 effort=10 velocity=10
- joint head: origin xyz=-0.00204165 -0 0.126 rpy=0 0 1.5708 -> xyz=0.01295835 0 0.126 rpy=0 0 1.5708
- joint left_foot_frame: origin xyz=-0 -0.023 0.042 rpy=-1.5708 -1.5708 0 -> xyz=-0 -0.0265 0.042 rpy=-1.5708 -1.5708 0
- joint left_hip_roll: limit lower=-0.610865 upper=0.610865 effort=10 velocity=10 -> lower=-0.436332 upper=0.436332 effort=10 velocity=10; origin xyz=0.02 0 -0.0214 rpy=-1.5708 -0 1.5708 -> xyz=0.0375 0 -0.0214 rpy=-1.5708 -0 1.5708
- joint right_foot_frame: origin xyz=-0 -0.023 0.042 rpy=-1.5708 -1.5708 0 -> xyz=-0 -0.0265 0.042 rpy=-1.5708 -1.5708 0
- joint right_hip_roll: limit lower=-0.610865 upper=0.610865 effort=10 velocity=10 -> lower=-0.436332 upper=0.436332 effort=10 velocity=10; origin xyz=-0.02 0 -0.0214 rpy=-1.5708 -0 -1.5708 -> xyz=-0.0375 0 -0.0214 rpy=-1.5708 -0 -1.5708
